Commit message: 修改了机器人laser的发布频率和质量以及摩擦力参数，使得小车能平滑的在room内运动和转向，并扫描了整个地图，利用navi2生成了map.yaml文件便于后续进行自动导航

File: chapter7/chapter7_ws/src/fishbot_description/urdf/fishbot/actuator/caster.urdf.xacro (robot description, xacro)
@@ -2,14 +2,14 @@
 <robot xmlns:xacro="http://www.ros.org/wiki/xacro" >
 <xacro:include filename="$(find fishbot_description)/urdf/fishbot/common_inertia.xacro"/>
-    <xacro:macro name="wheel_xacro" params="wheel_name xyz">
+    <xacro:macro name="caster_xacro" params="caster_name xyz">
         <!-- 机器人的IMU（Inertial Measurement Unit）部件，惯性测量单元 -->
-        <link name="${wheel_name}_link">
+        <link name="${caster_name}_link">
             <!-- 部件的外观描述 -->
             <visual>
                 <!-- 沿着自己的几何中心的偏移和旋转 -->
-                <origin xyz="0.0 0.0 0.0" rpy="1.57079 0.0 0.0"/>
+                <origin xyz="0.0 0.0 0.0" rpy="0.0 0.0 0.0"/>
                 <!-- 几何形状 -->
                 <geometry>
-                    <cylinder radius="0.0325" length="0.04"/>
+                    <sphere radius="0.016"/>
                 </geometry>
                 <!-- 材质颜色 -->
@@ -21,8 +21,8 @@
             <collision>
                 <!-- 沿着自己的几何中心的偏移和旋转 -->
-                <origin xyz="0.0 0.0 0.0" rpy="1.57079 0.0 0.0"/>
+                <origin xyz="0.0 0.0 0.0" rpy="0.0 0.0 0.0"/>
                 <!-- 几何形状 -->
                 <geometry>
-                    <cylinder radius="0.0325" length="0.04"/>
+                    <sphere radius="0.016"/>
                 </geometry>
                 <!-- 材质颜色 -->
@@ -32,23 +32,22 @@
                 </material>
             </collision>
-            <xacro:cylinder_inertia m ="0.05" r="0.0325" h="0.04" />
+            <xacro:sphere_inertia m ="0.1" r="0.016" />
         </link>
         <!-- 机器人的关节 Joint，用于组合机器人的部件 -->
-        <joint name="${wheel_name}_joint" type="continuous">
+        <joint name="${caster_name}_joint" type="fixed">
             <origin xyz="${xyz}" rpy="0.0 0.0 0.0"/>
-            <axis xyz="0.0 1.0 0.0"/>
             <parent link="base_link"/>
-            <child link="${wheel_name}_link"/>
+            <child link="${caster_name}_link"/>
         </joint>
         <!-- Gazebo 配置 -->
-        <gazebo reference='${wheel_name}_link'>
+        <gazebo reference='${caster_name}_link'>
             <!--mu1表示切向的阻尼系数  -->
-            <mu1 value= "20.0" />
+            <mu1 value= "0.01" />
             <!--mu2表示法向的阻尼系数  -->
-            <mu2 value= "20.0" />
+            <mu2 value= "0.01" />
             <!--kp表示接触的刚度系数  -->
-            <kp value= "1000000000.0" />
+            <kp value= "1000000.0" />
             <!--kd表示接触的阻尼系数  -->
-            <kd value= "1.0" />
+            <kd value= "100.0" />
         </gazebo>
     </xacro:macro>

File: chapter7/chapter7_ws/src/fishbot_description/urdf/fishbot/base.urdf.xacro (robot description, xacro)
@@ -1,8 +1,10 @@
 <?xml version="1.0"?>
 <robot xmlns:xacro="http://www.ros.org/wiki/xacro" >
+<!-- 引入对应转动惯量矩阵的宏文件 -->
 <xacro:include filename="$(find fishbot_description)/urdf/fishbot/common_inertia.xacro"/>
-    <xacro:macro name="caster_xacro" params="caster_name xyz">
-        <!-- 机器人的IMU（Inertial Measurement Unit）部件，惯性测量单元 -->
-        <link name="${caster_name}_link">
+    <xacro:macro name="base_xacro" params="length radius">
+        <link name="base_footprint" />
+        <!-- 机器人的身体部分 -->
+        <link name="base_link">
             <!-- 部件的外观描述 -->
             <visual>
@@ -11,10 +13,11 @@
                 <!-- 几何形状 -->
                 <geometry>
-                    <sphere radius="0.016"/>
+                    <!-- 单位是m -->
+                    <cylinder radius="${radius}" length="${length}"/>
                 </geometry>
                 <!-- 材质颜色 -->
-                <material name = "yellow">
+                <material name = "white">
                     <!-- rgb表示红绿蓝，范围为0～1，a表示透明度 -->
-                    <color rgba="1.0 1.0 0.0 0.8"/>
+                    <color rgba="1.0 1.0 1.0 0.5"/>
                 </material>
             </visual>
@@ -24,19 +27,19 @@
                 <!-- 几何形状 -->
                 <geometry>
-                    <sphere radius="0.016"/>
+                    <!-- 单位是m -->
+                    <cylinder radius="${radius}" length="${length}"/>
                 </geometry>
                 <!-- 材质颜色 -->
-                <material name = "yellow">
+                <material name = "white">
                     <!-- rgb表示红绿蓝，范围为0～1，a表示透明度 -->
-                    <color rgba="1.0 1.0 0.0 0.8"/>
+                    <color rgba="1.0 1.0 1.0 0.5"/>
                 </material>
             </collision>
-            <xacro:sphere_inertia m ="0.05" r="0.016" />
+            <xacro:cylinder_inertia m ="1.0" r="${radius}" h="${length}" />
         </link>
-        <!-- 机器人的关节 Joint，用于组合机器人的部件 -->
-        <joint name="${caster_name}_joint" type="fixed">
-            <origin xyz="${xyz}" rpy="0.0 0.0 0.0"/>
-            <parent link="base_link"/>
-            <child link="${caster_name}_link"/>
+        <joint name="joint_name" type="fixed">
+            <origin xyz="0.0 0.0 ${length/2.0 +0.03205}" rpy="0.0 0.0 0.0"/>
+            <parent link="base_footprint"/>
+            <child link="base_link"/>
         </joint>
     </xacro:macro>

File: chapter7/chapter7_ws/src/fishbot_description/urdf/fishbot/fishbot.urdf.xacro (robot description, xacro)
@@ -20,6 +20,6 @@
 <xacro:wheel_xacro  wheel_name = "left_wheel" xyz = "0 0.10 -0.06" />
 <xacro:wheel_xacro  wheel_name = "right_wheel" xyz = "0 -0.10 -0.06" />
-<xacro:caster_xacro  caster_name = "front_caster" xyz = "0.08 0 -0.06" />
-<xacro:caster_xacro  caster_name = "back_caster" xyz = "-0.08 0 -0.06" />
+<xacro:caster_xacro  caster_name = "front_caster" xyz = "0.08 0 -0.076" />
+<xacro:caster_xacro  caster_name = "back_caster" xyz = "-0.08 0 -0.076" />
 <!-- <xacro:gazebo_control_plugin /> -->
 <!-- 防止ros2_control插件和gazebo插件控制两轮差速硬件冲突，因此注释掉gazebo_control 插件 -->

File: chapter7/chapter7_ws/src/fishbot_description/urdf/fishbot/plugins/gazebo_sensor_plugin.xacro (robot description, xacro)
@@ -123,5 +123,6 @@
         </plugin>
         <always_on>true</always_on>
-        <update_rate>10</update_rate>
+        <!-- 原10 -->
+        <update_rate>100</update_rate>
         <camera name="camera">
             <!-- 水平视角的fov配置 -->

File: chapter7/chapter7_ws/src/fishbot_description/urdf/fishbot/sensor/camera.urdf.xacro (robot description, xacro)
@@ -2,7 +2,6 @@
 <robot xmlns:xacro="http://www.ros.org/wiki/xacro" >
 <xacro:include filename="$(find fishbot_description)/urdf/fishbot/common_inertia.xacro"/>
-    <xacro:macro name="imu_xacro" params="xyz">
-        <!-- 机器人的IMU（Inertial Measurement Unit）部件，惯性测量单元 -->
-        <link name="imu_link">
+    <xacro:macro name="camera_xacro" params="xyz">
+        <link name="camera_link">
             <!-- 部件的外观描述 -->
             <visual>
@@ -11,5 +10,5 @@
                 <!-- 几何形状 -->
                 <geometry>
-                        <box size="0.02 0.02 0.02"/>
+                        <box size="0.02 0.10 0.02"/>
                 </geometry>
                 <!-- 材质颜色 -->
@@ -24,5 +23,5 @@
                 <!-- 几何形状 -->
                 <geometry>
-                        <box size="0.02 0.02 0.02"/>
+                        <box size="0.02 0.10 0.02"/>
                 </geometry>
                 <!-- 材质颜色 -->
@@ -32,11 +31,20 @@
                 </material>
             </collision>
-            <xacro:box_inertia m ="0.05" w="0.02" h="0.02" d="0.02"  />
+            <xacro:box_inertia m ="0.01" w="0.02" h="0.10" d="0.02"  />
+        </link>
+        <link name="camera_optical_link">
+            <!-- 深度相机和彩色相机结合获取三维坐标数据 -->
+            <!-- 一般深度相机的面向方向为Z轴，因此需要使用虚拟部件来转换坐标系,将base_link坐标系转换为z轴向前的坐标系 -->
         </link>
         <!-- 机器人的关节 Joint，用于组合机器人的部件 -->
-        <joint name="imu_joint" type="fixed">
+        <joint name="camera_joint" type="fixed">
             <origin xyz="${xyz}" rpy="0.0 0.0 0.0"/>
             <parent link="base_link"/>
-            <child link="imu_link"/>
+            <child link="camera_link"/>
+        </joint>
+        <joint name="camera_optical_joint" type="fixed">
+            <origin xyz="0 0 0 " rpy="${-pi/2} 0.0 ${-pi/2}"/>
+            <parent link="camera_link"/>
+            <child link="camera_optical_link"/>
         </joint>
     </xacro:macro>

File: chapter7/chapter7_ws/src/fishbot_description/urdf/fishbot/sensor/imu.urdf.xacro (robot description, xacro)
@@ -2,6 +2,7 @@
 <robot xmlns:xacro="http://www.ros.org/wiki/xacro" >
 <xacro:include filename="$(find fishbot_description)/urdf/fishbot/common_inertia.xacro"/>
-    <xacro:macro name="camera_xacro" params="xyz">
-        <link name="camera_link">
+    <xacro:macro name="imu_xacro" params="xyz">
+        <!-- 机器人的IMU（Inertial Measurement Unit）部件，惯性测量单元 -->
+        <link name="imu_link">
             <!-- 部件的外观描述 -->
             <visual>
@@ -10,5 +11,5 @@
                 <!-- 几何形状 -->
                 <geometry>
-                        <box size="0.02 0.10 0.02"/>
+                        <box size="0.02 0.02 0.02"/>
                 </geometry>
                 <!-- 材质颜色 -->
@@ -23,5 +24,5 @@
                 <!-- 几何形状 -->
                 <geometry>
-                        <box size="0.02 0.10 0.02"/>
+                        <box size="0.02 0.02 0.02"/>
                 </geometry>
                 <!-- 材质颜色 -->
@@ -31,20 +32,11 @@
                 </material>
             </collision>
-            <xacro:box_inertia m ="0.1" w="0.02" h="0.10" d="0.02"  />
-        </link>
-        <link name="camera_optical_link">
-            <!-- 深度相机和彩色相机结合获取三维坐标数据 -->
-            <!-- 一般深度相机的面向方向为Z轴，因此需要使用虚拟部件来转换坐标系,将base_link坐标系转换为z轴向前的坐标系 -->
+            <xacro:box_inertia m ="0.01" w="0.02" h="0.02" d="0.02"  />
         </link>
         <!-- 机器人的关节 Joint，用于组合机器人的部件 -->
-        <joint name="camera_joint" type="fixed">
+        <joint name="imu_joint" type="fixed">
             <origin xyz="${xyz}" rpy="0.0 0.0 0.0"/>
             <parent link="base_link"/>
-            <child link="camera_link"/>
-        </joint>
-        <joint name="camera_optical_joint" type="fixed">
-            <origin xyz="0 0 0 " rpy="${-pi/2} 0.0 ${-pi/2}"/>
-            <parent link="camera_link"/>
-            <child link="camera_optical_link"/>
+            <child link="imu_link"/>
         </joint>
     </xacro:macro>

File: chapter7/chapter7_ws/src/fishbot_description/urdf/fishbot/sensor/laser.urdf.xacro (robot description, xacro)
@@ -63,5 +63,5 @@
                 </material>
             </collision>
-            <xacro:cylinder_inertia m ="0.10" r="0.02" h="0.02" />
+            <xacro:cylinder_inertia m ="0.01" r="0.02" h="0.02" />
         </link>
         <!-- 机器人的关节 Joint，用于组合机器人的部件 -->
