Commit message: 完成urdf小车建模和joint状态静态发布，能在rqt-tf-tree中看到话题发布

File: chapter9/fishbot_ws/src/fishbot_description/urdf/fishbot.urdf (robot description, URDF)
Before this commit: robot fishbot, 2 links, 0 joints
Links:
- added link laser_link; visual cylinder length=0.02 radius=0.02
Joints:
- added joint base_joint: type fixed, parent base_footprint, child base_link, origin xyz=0.0 0.0 0.076 rpy=0.0 0.0 0.0
- added joint laser_joint: type fixed, parent base_link, child laser_link, origin xyz=-0.10 0.0 0.075 rpy=0.0 0.0 0.0
